Commit message: removing robot base tf due to tf tree update problems: trunk tf would have two parents (base and odom)

File: xacro/gazebo.xacro (robot description, xacro)
@@ -13,5 +13,5 @@
             <frequency>10</frequency>
             <plot>
-                <link>base</link>
+                <link>trunk</link>
                 <pose>0 0 0 0 0 0</pose>
                 <material>Gazebo/Yellow</material>
@@ -121,8 +121,8 @@
         </visual>
     </gazebo>
-    <gazebo reference="base">
+    <!-- <gazebo reference="base">
         <material>Gazebo/Green</material>
         <turnGravityOff>false</turnGravityOff>
-    </gazebo>
+    </gazebo> -->
     <gazebo reference="trunk">
         <mu1>0.2</mu1>

File: xacro/robot.xacro (robot description, xacro)
@@ -13,7 +13,8 @@
             <origin rpy="0 0 0" xyz="0 0 0"/>
             <parent link="world"/>
-            <child link="base"/>
+            <child link="trunk"/>
         </joint>
     </xacro:if>
+<!--
     <link name="base">
         <visual>
@@ -28,5 +29,5 @@
         <parent link="base"/>
         <child link="trunk"/>
-    </joint>
+    </joint> -->
     <link name="trunk">
         <visual>

Commit message: Added plugin and configuration files

File: xacro/gazebo.xacro (robot description, xacro)
@@ -1,21 +1,45 @@
 <?xml version="1.0"?>
-<robot>
+<robot xmlns:xacro="http://www.ros.org/wiki/xacro">
+    <!-- Define the ROS version as a property -->
+    <xacro:property name="ros_version" value="$(env ROS_VERSION)" />
     <!-- ros_control plugin -->
     <gazebo>
-        <plugin name="gazebo_ros_control" filename="libgazebo_ros_control.so">
-            <robotNamespace>/b1_gazebo</robotNamespace>
-            <robotSimType>gazebo_ros_control/DefaultRobotHWSim</robotSimType>
-        </plugin>
+        <xacro:if value="${ros_version == 1}">
+            <plugin name="gazebo_ros_control" filename="libgazebo_ros_control.so">
+                <robotNamespace>/b1_gazebo</robotNamespace>
+                <robotSimType>gazebo_ros_control/DefaultRobotHWSim</robotSimType>
+            </plugin>
+        </xacro:if>
+        <xacro:if value="${ros_version == 2}">
+            <plugin filename="libgazebo_ros2_control.so" name="gazebo_ros2_control">
+            <parameters>$(find b1_description)/config/ros_control/ros_control.yaml</parameters>
+          </plugin>
+        </xacro:if>
     </gazebo>
     <!-- Show the trajectory of trunk center. -->
     <gazebo>
-        <plugin name="3dplot" filename="libLinkPlot3DPlugin.so">
-            <frequency>10</frequency>
-            <plot>
-                <link>trunk</link>
-                <pose>0 0 0 0 0 0</pose>
-                <material>Gazebo/Yellow</material>
-            </plot>
-        </plugin>
+        <xacro:if value="${ros_version == 1}">
+            <plugin name="3dplot" filename="libLinkPlot3DPlugin.so">
+                <frequency>10</frequency>
+                <plot>
+                    <link>base</link>
+                    <pose>0 0 0 0 0 0</pose>
+                    <material>Gazebo/Yellow</material>
+                </plot>
+            </plugin>
+        </xacro:if>
+        <xacro:if value="${ros_version == 2}">
+            <plugin name="p3d_base_controller" filename="libgazebo_ros_p3d.so">
+              <ros>
+                  <argument>odom:=odom/ground_truth</argument>
+              </ros>
+              <body_name>base</body_name>
+              <frame_name>world</frame_name>
+              <update_rate>10.0</update_rate>
+              <xyz_offset>0 0 0</xyz_offset>
+              <rpy_offset>0 0 0</rpy_offset>
+              <gaussian_noise>0.01</gaussian_noise>
+          </plugin>
+        </xacro:if>
     </gazebo>
     <!-- Show the trajectory of foot. You can add another trajectory about another foot. -->
@@ -31,8 +55,16 @@
     </gazebo> -->
     <gazebo>
-        <plugin filename="libgazebo_ros_force.so" name="gazebo_ros_force">
-            <bodyName>trunk</bodyName>
-            <topicName>/apply_force/trunk</topicName>
-        </plugin>
+        <xacro:if value="${ros_version == 1}">
+            <plugin filename="libgazebo_ros_force.so" name="gazebo_ros_force">
+                <bodyName>trunk</bodyName>
+                <topicName>/apply_force/trunk</topicName>
+            </plugin>
+        </xacro:if>
+        <xacro:if value="${ros_version == 2}">
+            <plugin filename="libgazebo_ros_force.so" name="gazebo_ros_force">
+                <link_name>base</link_name>
+                <topicName>/apply_force/trunk</topicName>
+            </plugin>
+        </xacro:if>
     </gazebo>
     <gazebo reference="imu_link">

File: xacro/leg.xacro (robot description, xacro)
@@ -58,5 +58,5 @@
                 </xacro:if>
                 <geometry>
-                    <mesh filename="package://b1_description/meshes/hip.dae" scale="1 1 1"/>
+                    <mesh filename="file://$(find b1_description)/meshes/hip.dae" scale="1 1 1"/>
                 </geometry>
                 <material name="orange"/>
@@ -118,8 +118,8 @@
                 <geometry>
                     <xacro:if value="${mirror_dae == True}">
-                        <mesh filename="package://b1_description/meshes/thigh.dae" scale="1 1 1"/>
+                        <mesh filename="file://$(find b1_description)/meshes/thigh.dae" scale="1 1 1"/>
                     </xacro:if>
                     <xacro:if value="${mirror_dae == False}">
-                        <mesh filename="package://b1_description/meshes/thigh_mirror.dae" scale="1 1 1"/>
+                        <mesh filename="file://$(find b1_description)/meshes/thigh_mirror.dae" scale="1 1 1"/>
                     </xacro:if>
                 </geometry>
@@ -181,5 +181,5 @@
                 <origin rpy="0 0 0" xyz="0 0 0"/>
                 <geometry>
-                    <mesh filename="package://b1_description/meshes/calf.dae" scale="1 1 1"/>
+                    <mesh filename="file://$(find b1_description)/meshes/calf.dae" scale="1 1 1"/>
                 </geometry>
                 <material name="orange"/>
@@ -251,4 +251,31 @@
         </link>
         <xacro:leg_transmission name="${name}"/>
+        <xacro:if value="${ros_version == 2}">
+            <ros2_control name="${name}" type="system">
+                <hardware>
+                    <plugin>gazebo_ros2_control/GazeboSystem</plugin>
+                </hardware>
+                <joint name="${name}_hip_joint">
+                    <command_interface name="effort"/>
+                    <state_interface name="position"/>
+                    <state_interface name="velocity"/>
+                </joint>
+                <joint name="${name}_thigh_joint">
+                    <command_interface name="effort"/>
+                    <state_interface name="position"/>
+                    <state_interface name="velocity"/>
+                </joint>
+                <joint name="${name}_calf_joint">
+                    <command_interface name="effort"/>
+                    <state_interface name="position"/>
+                    <state_interface name="velocity"/>
+                </joint>
+                <joint name="${name}_foot_fixed">
+                    <command_interface name="effort"/>
+                    <state_interface name="position"/>
+                    <state_interface name="velocity"/>
+                </joint>
+            </ros2_control>
+        </xacro:if>
     </xacro:macro>
 </robot>

File: xacro/robot.xacro (robot description, xacro)
@@ -1,4 +1,5 @@
 <?xml version="1.0"?>
 <robot name="b1_description" xmlns:xacro="http://www.ros.org/wiki/xacro">
+    <xacro:arg name="DEBUG" default="false"/>
     <xacro:include filename="$(find b1_description)/xacro/const.xacro"/>
     <xacro:include filename="$(find b1_description)/xacro/materials.xacro"/>
@@ -34,5 +35,5 @@
             <origin rpy="0 0 0" xyz="0 0 0"/>
             <geometry>
-                <mesh filename="package://b1_description/meshes/trunk.dae" scale="1 1 1"/>
+                <mesh filename="file://$(find b1_description)/meshes/trunk.dae" scale="1 1 1"/>
             </geometry>
             <material name="orange"/>
@@ -47,5 +48,5 @@
             <origin rpy="0 0 0" xyz="0 0 0"/>
             <geometry>
-                <mesh filename="package://b1_description/meshes/trunk.dae" scale="1 1 1"/>
+                <mesh filename="file://$(find b1_description)/meshes/trunk.dae" scale="1 1 1"/>
             </geometry>
         </collision> -->

Commit message: Minor

File: xacro/gazebo.xacro (robot description, xacro)
@@ -13,5 +13,6 @@
         <xacro:if value="${ros_version == 2}">
             <plugin filename="libgazebo_ros2_control.so" name="gazebo_ros2_control">
-            <parameters>$(find b1_description)/config/ros_control/ros_control.yaml</parameters>
+                <parameters>$(find b1_description)/config/ros_control/ros_control.yaml</parameters>
+                <controlPeriod>0.001</controlPeriod>
           </plugin>
         </xacro:if>
@@ -23,5 +24,5 @@
                 <frequency>10</frequency>
                 <plot>
-                    <link>base</link>
+                    <link>trunk</link>
                     <pose>0 0 0 0 0 0</pose>
                     <material>Gazebo/Yellow</material>
@@ -34,5 +35,5 @@
                   <argument>odom:=odom/ground_truth</argument>
               </ros>
-              <body_name>base</body_name>
+              <body_name>trunk</body_name>
               <frame_name>world</frame_name>
               <update_rate>10.0</update_rate>
