Commit message: Modified xacro file to work with ignition

File: xacro/gazebo.xacro (robot description, xacro)
@@ -3,4 +3,6 @@
     <!-- Define the ROS version as a property -->
     <xacro:property name="ros_version" value="$(env ROS_VERSION)" />
+    <xacro:arg name="ign" default="false"/>
+    <xacro:property name="ign" value="$(arg ign)"/>
     <!-- ros_control plugin -->
     <gazebo>
@@ -12,12 +14,22 @@
         </xacro:if>
         <xacro:if value="${ros_version == 2}">
-            <plugin filename="libgazebo_ros2_control.so" name="gazebo_ros2_control">
-                <parameters>$(find b1_description)/config/ros_control/ros_control.yaml</parameters>
-                <controlPeriod>0.001</controlPeriod>
-          </plugin>
+            <xacro:if value="${ign}">
+                <plugin filename="ign_ros2_control-system" name="ign_ros2_control::IgnitionROS2ControlPlugin">
+                    <robot_param>robot_description</robot_param>
+                    <robot_param_node>robot_state_publisher</robot_param_node>
+                    <parameters>$(find b1_description)/config/ros_control/ros_control.yaml</parameters>
+                    <!-- <controlPeriod>0.001</controlPeriod> -->
+                </plugin>
+            </xacro:if>
+            <xacro:unless value="${ign}">
+                <plugin filename="libgazebo_ros2_control.so" name="gazebo_ros2_control">
+                    <parameters>$(find b1_description)/config/ros_control/ros_control.yaml</parameters>
+                    <controlPeriod>0.001</controlPeriod>
+                </plugin>
+            </xacro:unless>
         </xacro:if>
     </gazebo>
     <!-- Show the trajectory of trunk center. -->
-    <gazebo>
+    <!-- <gazebo>
         <xacro:if value="${ros_version == 1}">
             <plugin name="3dplot" filename="libLinkPlot3DPlugin.so">
@@ -43,5 +55,5 @@
           </plugin>
         </xacro:if>
-    </gazebo>
+    </gazebo> -->
     <!-- Show the trajectory of foot. You can add another trajectory about another foot. -->
     <!-- <gazebo>
@@ -55,5 +67,5 @@
         </plugin>
     </gazebo> -->
-    <gazebo>
+    <!-- <gazebo>
         <xacro:if value="${ros_version == 1}">
             <plugin filename="libgazebo_ros_force.so" name="gazebo_ros_force">
@@ -87,7 +99,7 @@
             <pose>0 0 0 0 0 0</pose>
         </sensor>
-    </gazebo>
+    </gazebo> -->
     <!-- Foot contacts. -->
-    <gazebo reference="FR_calf">
+    <!-- <gazebo reference="FR_calf">
         <sensor name="FR_foot_contact" type="contact">
         <update_rate>100</update_rate>
@@ -124,7 +136,7 @@
         </contact>
         </sensor>
-    </gazebo>
+    </gazebo> -->
     <!-- Visualization of Foot contacts. -->
-    <gazebo reference="FR_foot">
+    <!-- <gazebo reference="FR_foot">
         <visual>
             <plugin name="drawForcePlugin" filename="libunitreeDrawForcePlugin.so">
@@ -153,5 +165,5 @@
             </plugin>
         </visual>
-    </gazebo>
+    </gazebo> -->
     <!-- <gazebo reference="base">
         <material>Gazebo/Green</material>
@@ -167,10 +179,14 @@
         <mu1>0.2</mu1>
         <mu2>0.2</mu2>
-        <material>Gazebo/White</material>
+        <xacro:unless value="${ign}">
+            <material>Gazebo/White</material>
+        </xacro:unless>
     </gazebo>
     <gazebo reference="imu_link">
         <mu1>0.2</mu1>
         <mu2>0.2</mu2>
-        <material>Gazebo/Red</material>
+        <xacro:unless value="${ign}">
+            <material>Gazebo/Red</material>
+        </xacro:unless>
     </gazebo>
     <!-- FL leg -->
@@ -178,5 +194,7 @@
         <mu1>0.2</mu1>
         <mu2>0.2</mu2>
-        <material>Gazebo/DarkGrey</material>
+        <xacro:unless value="${ign}">
+            <material>Gazebo/DarkGrey</material>
+        </xacro:unless>
     </gazebo>
     <gazebo reference="FL_thigh">
@@ -184,5 +202,7 @@
         <mu2>0.2</mu2>
         <self_collide>1</self_collide>
-        <material>Gazebo/DarkGrey</material>
+        <xacro:unless value="${ign}">
+            <material>Gazebo/DarkGrey</material>
+        </xacro:unless>
         <kp  value="1000000.0"/>
         <kd  value="1.0"/>
@@ -197,5 +217,7 @@
         <mu2>0.6</mu2>
         <self_collide>1</self_collide>
-        <material>Gazebo/DarkGrey</material>
+        <xacro:unless value="${ign}">
+            <material>Gazebo/DarkGrey</material>
+        </xacro:unless>
         <kp  value="1000000.0"/>
         <kd  value="1.0"/>
@@ -205,5 +227,7 @@
         <mu1>0.2</mu1>
         <mu2>0.2</mu2>
-        <material>Gazebo/DarkGrey</material>
+        <xacro:unless value="${ign}">
+            <material>Gazebo/DarkGrey</material>
+        </xacro:unless>
     </gazebo>
     <gazebo reference="FR_thigh">
@@ -211,5 +235,7 @@
         <mu2>0.2</mu2>
         <self_collide>1</self_collide>
-        <material>Gazebo/DarkGrey</material>
+        <xacro:unless value="${ign}">
+            <material>Gazebo/DarkGrey</material>
+        </xacro:unless>
         <kp  value="1000000.0"/>
         <kd  value="1.0"/>
@@ -224,5 +250,7 @@
         <mu2>0.6</mu2>
         <self_collide>1</self_collide>
-        <material>Gazebo/DarkGrey</material>
+        <xacro:unless value="${ign}">
+            <material>Gazebo/DarkGrey</material>
+        </xacro:unless>
         <kp  value="1000000.0"/>
         <kd  value="1.0"/>
@@ -232,5 +260,7 @@
         <mu1>0.2</mu1>
         <mu2>0.2</mu2>
-        <material>Gazebo/DarkGrey</material>
+        <xacro:unless value="${ign}">
+            <material>Gazebo/DarkGrey</material>
+        </xacro:unless>
     </gazebo>
     <gazebo reference="RL_thigh">
@@ -238,5 +268,7 @@
         <mu2>0.2</mu2>
         <self_collide>1</self_collide>
-        <material>Gazebo/DarkGrey</material>
+        <xacro:unless value="${ign}">
+            <material>Gazebo/DarkGrey</material>
+        </xacro:unless>
         <kp  value="1000000.0"/>
         <kd  value="1.0"/>
@@ -251,5 +283,7 @@
         <mu2>0.6</mu2>
         <self_collide>1</self_collide>
-        <material>Gazebo/DarkGrey</material>
+        <xacro:unless value="${ign}">
+            <material>Gazebo/DarkGrey</material>
+        </xacro:unless>
         <kp  value="1000000.0"/>
         <kd  value="1.0"/>
@@ -259,5 +293,7 @@
         <mu1>0.2</mu1>
         <mu2>0.2</mu2>
-        <material>Gazebo/DarkGrey</material>
+        <xacro:unless value="${ign}">
+            <material>Gazebo/DarkGrey</material>
+        </xacro:unless>
     </gazebo>
     <gazebo reference="RR_thigh">
@@ -265,5 +301,7 @@
         <mu2>0.2</mu2>
         <self_collide>1</self_collide>
-        <material>Gazebo/DarkGrey</material>
+        <xacro:unless value="${ign}">
+            <material>Gazebo/DarkGrey</material>
+        </xacro:unless>
         <kp  value="1000000.0"/>
         <kd  value="1.0"/>
@@ -278,5 +316,7 @@
         <mu2>0.6</mu2>
         <self_collide>1</self_collide>
-        <material>Gazebo/DarkGrey</material>
+        <xacro:unless value="${ign}">
+            <material>Gazebo/DarkGrey</material>
+        </xacro:unless>
         <kp  value="1000000.0"/>
         <kd  value="1.0"/>

File: xacro/leg.xacro (robot description, xacro)
@@ -1,4 +1,7 @@
 <?xml version="1.0"?>
 <robot xmlns:xacro="http://www.ros.org/wiki/xacro">
+    <xacro:property name="ros_version" value="$(env ROS_VERSION)" />
+    <xacro:arg name="ign" default="false"/>
+    <xacro:property name="ign" value="$(arg ign)"/>
     <xacro:include filename="$(find b1_description)/xacro/transmission.xacro"/>
     <xacro:macro name="leg" params="name mirror mirror_dae front_hind front_hind_dae">
@@ -60,5 +63,5 @@
                     <mesh filename="file://$(find b1_description)/meshes/hip.dae" scale="1 1 1"/>
                 </geometry>
-                <material name="orange"/>
+                <material name="white"/>
             </visual>
             <collision>
@@ -83,5 +86,5 @@
                     <cylinder length="0.02" radius="0.05"/>
                 </geometry>
-                <material name="green"/>
+                <material name="steel_grey"/>
             </visual>
             <!-- <collision>
@@ -124,5 +127,5 @@
                     </xacro:if>
                 </geometry>
-                <material name="orange"/>
+                <material name="steel_grey"/>
             </visual>
             <collision>
@@ -147,5 +150,5 @@
                     <cylinder length="0.02" radius="0.05"/>
                 </geometry>
-                <material name="green"/>
+                <material name="steel_grey"/>
             </visual>
             <!-- <collision>
@@ -183,5 +186,5 @@
                     <mesh filename="file://$(find b1_description)/meshes/calf.dae" scale="1 1 1"/>
                 </geometry>
-                <material name="orange"/>
+                <material name="white"/>
             </visual>
             <collision>
@@ -206,5 +209,5 @@
                     <cylinder length="0.02" radius="0.05"/>
                 </geometry>
-                <material name="green"/>
+                <material name="steel_grey"/>
             </visual>
             <!-- <collision>
@@ -234,5 +237,5 @@
                     <sphere radius="${foot_radius-0.01}"/>
                 </geometry>
-                <material name="green"/>
+                <material name="steel_grey"/>
             </visual>
             <collision>
@@ -252,29 +255,58 @@
         <xacro:leg_transmission name="${name}"/>
         <xacro:if value="${ros_version == 2}">
-            <ros2_control name="${name}" type="system">
-                <hardware>
-                    <plugin>gazebo_ros2_control/GazeboSystem</plugin>
-                </hardware>
-                <joint name="${name}_hip_joint">
-                    <command_interface name="effort"/>
-                    <state_interface name="position"/>
-                    <state_interface name="velocity"/>
-                </joint>
-                <joint name="${name}_thigh_joint">
-                    <command_interface name="effort"/>
-                    <state_interface name="position"/>
-                    <state_interface name="velocity"/>
-                </joint>
-                <joint name="${name}_calf_joint">
-                    <command_interface name="effort"/>
-                    <state_interface name="position"/>
-                    <state_interface name="velocity"/>
-                </joint>
-                <joint name="${name}_foot_fixed">
-                    <command_interface name="effort"/>
-                    <state_interface name="position"/>
-                    <state_interface name="velocity"/>
-                </joint>
-            </ros2_control>
+            <xacro:if value="${ign}">
+                <ros2_control name="${name}" type="system">
+                    <hardware>
+                        <plugin>ign_ros2_control/IgnitionSystem</plugin>
+                    </hardware>
+                    <joint name="${name}_hip_joint">
+                        <command_interface name="effort"/>
+                        <state_interface name="position"/>
+                        <state_interface name="velocity"/>
+                    </joint>
+                    <joint name="${name}_thigh_joint">
+                        <command_interface name="effort"/>
+                        <state_interface name="position"/>
+                        <state_interface name="velocity"/>
+                    </joint>
+                    <joint name="${name}_calf_joint">
+                        <command_interface name="effort"/>
+                        <state_interface name="position"/>
+                        <state_interface name="velocity"/>
+                    </joint>
+                    <joint name="${name}_foot_fixed">
+                        <command_interface name="effort"/>
+                        <state_interface name="position"/>
+                        <state_interface name="velocity"/>
+                    </joint>
+                </ros2_control>
+            </xacro:if>
+            <xacro:unless value="${ign}">
+                <ros2_control name="${name}" type="system">
+                    <hardware>
+                        <plugin>gazebo_ros2_control/GazeboSystem</plugin>
+                    </hardware>
+                    <joint name="${name}_hip_joint">
+                        <command_interface name="effort"/>
+                        <state_interface name="position"/>
+                        <state_interface name="velocity"/>
+                    </joint>
+                    <joint name="${name}_thigh_joint">
+                        <command_interface name="effort"/>
+                        <state_interface name="position"/>
+                        <state_interface name="velocity"/>
+                    </joint>
+                    <joint name="${name}_calf_joint">
+                        <command_interface name="effort"/>
+                        <state_interface name="position"/>
+                        <state_interface name="velocity"/>
+                    </joint>
+                    <joint name="${name}_foot_fixed">
+                        <command_interface name="effort"/>
+                        <state_interface name="position"/>
+                        <state_interface name="velocity"/>
+                    </joint>
+                </ros2_control>
+            </xacro:unless>
         </xacro:if>
     </xacro:macro>

File: xacro/materials.xacro (robot description, xacro)
@@ -1,4 +1,7 @@
 <?xml version="1.0"?>
-<robot>
+<robot xmlns:xacro="http://www.ros.org/wiki/xacro">
+	<material name="steel_grey">
+    	<color rgba="${113/255} ${121/255} ${126/255} 1.0"/>
+  	</material>
     <material name="black">
         <color rgba="0.0 0.0 0.0 1.0"/>

File: xacro/robot.xacro (robot description, xacro)
@@ -37,5 +37,5 @@
                 <mesh filename="file://$(find b1_description)/meshes/trunk.dae" scale="1 1 1"/>
             </geometry>
-            <material name="orange"/>
+            <material name="steel_grey"/>
         </visual>
         <collision>
@@ -97,5 +97,5 @@
     <xacro:if value="$(arg SENSORS)">
         <xacro:property name="LIDAR" value="true"/>
-        <xacro:property name="CAMERAS" value="true"/>
+        <xacro:property name="CAMERAS" value="false"/>
     </xacro:if>
     <xacro:include filename="$(find b1_description)/xacro/sensors.xacro"/>

Commit message: Added ignition foretrees plugin

File: xacro/gazebo.xacro (robot description, xacro)
@@ -31,5 +31,5 @@
     </gazebo>
     <!-- Show the trajectory of trunk center. -->
-    <!-- <gazebo>
+    <gazebo>
         <xacro:if value="${ros_version == 1}">
             <plugin name="3dplot" filename="libLinkPlot3DPlugin.so">
@@ -43,29 +43,33 @@
         </xacro:if>
         <xacro:if value="${ros_version == 2}">
-            <plugin name="p3d_base_controller" filename="libgazebo_ros_p3d.so">
-              <ros>
-                  <argument>odom:=odom/ground_truth</argument>
-              </ros>
-              <body_name>trunk</body_name>
-              <frame_name>world</frame_name>
-              <update_rate>10.0</update_rate>
-              <xyz_offset>0 0 0</xyz_offset>
-              <rpy_offset>0 0 0</rpy_offset>
-              <gaussian_noise>0.01</gaussian_noise>
-          </plugin>
-        </xacro:if>
-    </gazebo> -->
+            <xacro:unless value="${ign}">
+                <plugin name="p3d_base_controller" filename="libgazebo_ros_p3d.so">
+                    <ros>
+                        <argument>odom:=odom/ground_truth</argument>
+                    </ros>
+                    <body_name>trunk</body_name>
+                    <frame_name>world</frame_name>
+                    <update_rate>10.0</update_rate>
+                    <xyz_offset>0 0 0</xyz_offset>
+                    <rpy_offset>0 0 0</rpy_offset>
+                    <gaussian_noise>0.01</gaussian_noise>
+                </plugin>
+            </xacro:unless>
+        </xacro:if>
+    </gazebo>
     <!-- Show the trajectory of foot. You can add another trajectory about another foot. -->
-    <!-- <gazebo>
-        <plugin name="3dplot" filename="libLinkPlot3DPlugin.so">
-            <frequency>100</frequency>
-            <plot>
-                <link>FL_foot</link>
-                <pose>0 0 0 0 0 0</pose>
-                <material>Gazebo/Green</material>
-            </plot>
-        </plugin>
-    </gazebo> -->
-    <!-- <gazebo>
+    <xacro:unless value="${ign}">
+        <gazebo>
+            <plugin name="3dplot" filename="libLinkPlot3DPlugin.so">
+                <frequency>100</frequency>
+                <plot>
+                    <link>FL_foot</link>
+                    <pose>0 0 0 0 0 0</pose>
+                    <material>Gazebo/Green</material>
+                </plot>
+            </plugin>
+        </gazebo>
+    </xacro:unless>
+    <gazebo>
         <xacro:if value="${ros_version == 1}">
             <plugin filename="libgazebo_ros_force.so" name="gazebo_ros_force">
@@ -74,32 +78,61 @@
             </plugin>
         </xacro:if>
-        <xacro:if value="${ros_version == 2}">
-            <plugin filename="libgazebo_ros_force.so" name="gazebo_ros_force">
-                <link_name>base</link_name>
-                <topicName>/apply_force/trunk</topicName>
-            </plugin>
-        </xacro:if>
-    </gazebo>
-    <gazebo reference="imu_link">
-        <gravity>true</gravity>
-        <sensor name="imu_sensor" type="imu">
-            <always_on>true</always_on>
-            <update_rate>1000</update_rate>
-            <visualize>true</visualize>
-            <topic>__default_topic__</topic>
-            <plugin filename="libgazebo_ros_imu_sensor.so" name="imu_plugin">
-                <topicName>trunk_imu</topicName>
-                <bodyName>imu_link</bodyName>
-                <updateRateHZ>1000.0</updateRateHZ>
-                <gaussianNoise>0.0</gaussianNoise>
-                <xyzOffset>0 0 0</xyzOffset>
-                <rpyOffset>0 0 0</rpyOffset>
-                <frameName>imu_link</frameName>
-            </plugin>
-            <pose>0 0 0 0 0 0</pose>
-        </sensor>
-    </gazebo> -->
+        <xacro:unless value="${ign}">
+            <xacro:if value="${ros_version == 2}">
+                <plugin filename="libgazebo_ros_force.so" name="gazebo_ros_force">
+                    <link_name>base</link_name>
+                    <topicName>/apply_force/trunk</topicName>
+                </plugin>
+            </xacro:if>
+        </xacro:unless>
+    </gazebo>
+    <xacro:unless value="${ign}">
+        <gazebo reference="imu_link">
+            <gravity>true</gravity>
+            <sensor name="imu_sensor" type="imu">
+                <always_on>true</always_on>
+                <update_rate>1000</update_rate>
+                <visualize>true</visualize>
+                <topic>__default_topic__</topic>
+                <plugin filename="libgazebo_ros_imu_sensor.so" name="imu_plugin">
+                    <ros>
+                        <namespace>/imu</namespace>
+                        <argument>~/out:=data</argument>
+                    </ros>
+                    <topicName>trunk_imu</topicName>
+                    <bodyName>imu_link</bodyName>
+                    <updateRateHZ>1000.0</updateRateHZ>
+                    <gaussianNoise>0.0</gaussianNoise>
+                    <xyzOffset>0 0 0</xyzOffset>
+                    <rpyOffset>0 0 0</rpyOffset>
+                    <frameName>imu_link</frameName>
+                </plugin>
+                <pose>0 0 0 0 0 0</pose>
+            </sensor>
+        </gazebo>
+    </xacro:unless>
+    <xacro:if value="${ign}">
+        <gazebo reference="imu_link">
+            <gravity>true</gravity>
+            <sensor name="imu_sensor" type="imu">
+                <always_on>true</always_on>
+                <update_rate>50</update_rate>
+                <visualize>true</visualize>
+                <topic>/imu/data</topic>
+                <plugin filename="libignition-gazebo-imu-system.so" name="ignition::gazebo::systems::Imu">
+                    <topicName>trunk_imu</topicName>
+                    <bodyName>imu_link</bodyName>
+                    <updateRateHZ>50.0</updateRateHZ>
+                    <gaussianNoise>0.0</gaussianNoise>
+                    <xyzOffset>0 0 0</xyzOffset>
+                    <rpyOffset>0 0 0</rpyOffset>
+                    <frameName>imu_link</frameName>
+                </plugin>
+                <pose>0 0 0 0 0 0</pose>
+            </sensor>
+        </gazebo>
+    </xacro:if>
     <!-- Foot contacts. -->
-    <!-- <gazebo reference="FR_calf">
+    <gazebo reference="FR_calf">
         <sensor name="FR_foot_contact" type="contact">
         <update_rate>100</update_rate>
@@ -136,7 +169,7 @@
         </contact>
         </sensor>
-    </gazebo> -->
+    </gazebo>
     <!-- Visualization of Foot contacts. -->
-    <!-- <gazebo reference="FR_foot">
+    <gazebo reference="FR_foot">
         <visual>
             <plugin name="drawForcePlugin" filename="libunitreeDrawForcePlugin.so">
@@ -165,5 +198,5 @@
             </plugin>
         </visual>
-    </gazebo> -->
+    </gazebo>
     <!-- <gazebo reference="base">
         <material>Gazebo/Green</material>
