Commit message: adding frame for correct lidar configuration

File: xacro/sensors.xacro (robot description, xacro)
@@ -39,4 +39,10 @@
         </xacro:VLP-16>
     </xacro:if>
+    <link name="hesai_lidar"/>
+    <joint name="hesai_lidar_joint" type="fixed">
+            <parent link="lidar"/>
+            <child link="hesai_lidar"/>
+            <origin xyz="0 0 0" rpy="0 0 1.57"/>
+    </joint>
     <!-- Cameras -->
     <xacro:if value="${CAMERAS}">

Commit message: adding hesai lidar tf for real application

File: xacro/sensors.xacro (robot description, xacro)
@@ -38,4 +38,10 @@
             <origin xyz="0 0 0.025" rpy="0 0 0" />
         </xacro:VLP-16>
+        <link name="hesai_lidar"/>
+        <joint name="hesai_lidar_joint" type="fixed">
+                <parent link="lidar"/>
+                <child link="hesai_lidar"/>
+                <origin xyz="0 0 0" rpy="0 0 1.57"/>
+        </joint>
     </xacro:if>
     <!-- Cameras -->

Commit message: modified bug

File: xacro/sensors.xacro (robot description, xacro)
@@ -39,10 +39,4 @@
         </xacro:VLP-16>
     </xacro:if>
-    <link name="hesai_lidar"/>
-    <joint name="hesai_lidar_joint" type="fixed">
-            <parent link="lidar"/>
-            <child link="hesai_lidar"/>
-            <origin xyz="0 0 0" rpy="0 0 1.57"/>
-    </joint>
     <!-- Cameras -->
     <xacro:if value="${CAMERAS}">

Commit message: using hesai x16 lidar

File: xacro/sensors.xacro (robot description, xacro)
@@ -1,5 +1,5 @@
 <?xml version="1.0"?>
 <robot xmlns:xacro="http://www.ros.org/wiki/xacro">
-    <xacro:include filename="$(find sensors_description)/xacro/VLP-16.urdf.xacro"/>
+    <xacro:include filename="$(find sensors_description)/xacro/hesai_xt16.xacro"/>
     <xacro:include filename="$(find sensors_description)/xacro/realsense_d430.urdf.xacro" />
     <!-- Lidar -->
@@ -34,12 +34,12 @@
             <material>Gazebo/White</material>
         </gazebo>
-        <xacro:VLP-16 parent="lidar_mount" name="lidar" sim_ignition="true" topic="/lidar_points">
+        <xacro:hesai_xt16 parent="lidar_mount" name="lidar" sim_ignition="true" topic_name="/lidar">
             <origin xyz="0 0 0.025" rpy="0 0 0" />
-        </xacro:VLP-16>
+        </xacro:hesai_xt16>
         <link name="hesai_lidar"/>
         <joint name="hesai_lidar_joint" type="fixed">
-                <parent link="lidar"/>
-                <child link="hesai_lidar"/>
-                <origin xyz="0 0 0" rpy="0 0 1.57"/>
+            <parent link="lidar"/>
+            <child link="hesai_lidar"/>
+            <origin xyz="0 0 0" rpy="0 0 1.57"/>
         </joint>
     </xacro:if>
